File: interfaceB-robot.sch (EAGLE design)
At the start: 24 parts, among them IC1 LD117AS33TR, M1 ESP12Q

Commit message: added schematic
Other:
- note added: "Motor A connected to GPIO 16,14,12,13"
- note added: "Motor B connected to GPIO 4,5,0,2"
- note added: "Ultrasonic connected to ADC"
Changed lines of the file:
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@@
 <sheet>
 <plain>
+<text x="157.48" y="25.4" size="1.778" layer="91">Motor A connected to GPIO 16,14,12,13</text>
+<text x="157.48" y="22.86" size="1.778" layer="91">Motor B connected to GPIO 4,5,0,2</text>
+<text x="157.48" y="20.32" size="1.778" layer="91">Ultrasonic connected to ADC</text>
 </plain>
 <instances>
